File: autoplanter.sch (KiCad schematic (older format))
At the start: 77 parts, among them IC1 KST10MTF, IC2 KST10MTF, IC3 BME680, IC4 MCP73842T-840I_UN, J1 water, J2 USB_C_Receptacle_USB2.0, J3 Conn_01x10_Female, J4 Conn_01x02_Female, K1 Y14x-1C-xxDS, M1 Motor_DC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

Commit message: Fixed regurator and added low voltage safe circuit.
Parts:
- added J5: I2C Debug, Connector_PinSocket_2.54mm:PinSocket_1x02_P2.54mm_Vertical, symbol autoplanter-cache:Connector_Conn_01x02_Female
- added J6: external regurator, Connector_PinSocket_2.54mm:PinSocket_1x03_P2.54mm_Vertical, symbol autoplanter-cache:Connector_Conn_01x03_Female
- added J7: 12v regurator, Connector_PinHeader_2.54mm:PinHeader_1x03_P2.54mm_Vertical, symbol autoplanter-cache:Connector_Conn_01x03_Female
- added Q1: DMG2301L-7, SOT96P240X110-3N, symbol SamacSys_Parts:DMG2301L-7
- added Q3: 2SC2712-Y,LF, SOT95P260X140-3N, symbol SamacSys_Parts:2SC2712-Y,LF
- added R27, R28: 20k, Capacitor_SMD:C_1206_3216Metric, symbol Device:R_Small
- added R29: 10k, Capacitor_SMD:C_1206_3216Metric, symbol Device:R_Small
- added SW3: SW_DIP_x01, Button_Switch_THT:SW_E-Switch_EG1271_DPDT, symbol Switch:SW_DIP_x01
- added Z1: MM3Z6V2T1G, SOD2512X110N, symbol SamacSys_Parts:MM3Z6V2T1G
Connections:
- net +BATT: now also Q1.3; no longer D4.2 (A)
- net -BATT: now also J6.2 (Pin_2), J7.2 (Pin_2), Q3.2, R29.2
- net at IC3.3 (SDI), R12.2, U2.33 (IO21)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: now also J5.1 (Pin_1)
- net at IC3.4 (SCK), R13.2, U2.36 (IO22)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: now also J5.2 (Pin_2)
- net at BT1.1 (+), C11.1, IC4.9 (VBAT)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: now also SW3.1; no longer D4.1 (K)
- net at C10.1, D6.2 (A), IC4.2 (VDD)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: now also J7.1 (Pin_1); no longer D5.2 (A)
- net at C16.1, JP4.2, L1.1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: now also J6.1 (Pin_1)
- net at C14.1, D7.2 (K), PS1.2 (IN)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: now also J6.3 (Pin_3)
- new net: D5.2 (A), J7.3 (Pin_3)
- new net: D4.2 (A), Q1.2, R27.1, R28.1
- new net: R27.2, Z1.1
- new net: Q1.1, Q3.3, R28.2
- new net: Q3.1, R29.1, Z1.2
- new net: D4.1 (K), SW3.2
Other:
- moved on the sheet: BT1, D5, SC1
